File: pcb/Sitrep_PCB/sitrep_display.sch (EAGLE design)
At the start: 113 parts, among them Q1 2N3904, Q11 2N3904, Q12 2N3904, Q13 2N3904, Q2 2N3904, Q3 2N3904, Q4 2N3904, Q5 2N3904, Q6 2N3904, Q8 2N3904

Commit message: Updated PCB files
Parts:
- removed DECADE-COUNTER: 4017N, 40xx:4017N
- removed LED102, LED104, LED110, LED111, LED115, LED119, LED120, LED127, LED128, LED133, LED135, LED136, LED141, LED144, LED85, LED87, LED88, LED89, LED94, LED96: (no value), adafruit:LED5MM
- removed Q11: 2N3904, transistor-npn:2N3904
- removed U$1: PHOTON_WITH_HEADERS, Particle-Devices:PHOTON_WITH_HEADERS
- removed U$2: ARDUINOUNO, adafruit:ARDUINOUNO
- added IC1: 4017N, 40xx:4017N
- added JP2: (no value), pinhead:PINHD-1X7/90
- added LED1, LED10, LED11, LED2, LED20, LED21, LED22, LED30, LED31, LED32, LED4, LED41, LED42, LED56, LED66, LED67, LED71, LED72, LED9: (no value), adafruit:LED5MM
- added Q7: 2N3904, transistor-npn:2N3904
- R1, R2, R3, R4, R5, R6, R8: value 150 -> 1k; device adafruit:R-US_0207/2V -> resistor:R-US_0204/2V
- R11, R12, R13, R14, R16, R17, R18: value 1k -> 150; device resistor:R-US_0204/2V -> adafruit:R-US_0207/2V
- R15: value (none) -> 150; device resistor:R-US_0204/2V -> adafruit:R-US_0207/2V
- R7: value 150 -> (none); device adafruit:R-US_0207/2V -> resistor:R-US_0204/2V
- renumbered LED100 to LED35, LED101 to LED45, LED103 to LED70, LED105 to LED15, LED106 to LED26, LED107 to LED36, LED108 to LED46, LED109 to LED51, LED113 to LED5, LED114 to LED16, LED116 to LED37, LED117 to LED47, LED118 to LED52, LED121 to LED6, LED122 to LED17, LED123 to LED27, LED124 to LED38, LED125 to LED48, LED126 to LED53, LED129 to LED7, LED130 to LED18, LED131 to LED28, LED132 to LED39, LED134 to LED54, LED137 to LED8, LED138 to LED19, LED139 to LED29, LED140 to LED40, LED142 to LED55, LED143 to LED65, LED81 to LED12, LED82 to LED23, LED83 to LED33, LED84 to LED43, LED86 to LED68, LED90 to LED13, LED91 to LED24, LED92 to LED34, LED93 to LED44, LED95 to LED69, LED97 to LED3, LED98 to LED14, LED99 to LED25, Q12 to Q9, Q13 to Q10, SHIFT-REGISTER to IC2
Connections:
- removed net N$1: U$1.TX, U$2.D0
- removed net N$15: LED17.A
- removed net N$2: U$1.RX, U$2.D1
- removed net N$23: LED27.A
- removed net N$25: LED38.A
- removed net N$26: LED48.A
- removed net N$27: LED53.A
- removed net N$28: LED127.A
- removed net N$29: LED70.C
- removed net N$3: IC2A.RCK, U$2.D9
- removed net N$34: LED128.A
- removed net N$36: LED6.A
- removed net N$4: IC2A.SCK, U$2.D10
- removed net N$40: LED18.A
- removed net N$41: LED28.A
- removed net N$42: LED39.A
- removed net N$43: LED133.A
- removed net N$44: LED54.A
- removed net N$45: LED135.A
- removed net N$46: LED136.A
- removed net N$47: LED7.A
- removed net N$49: LED19.A
- removed net N$5: IC2A.SER, U$2.D11
- removed net N$50: LED29.A
- removed net N$51: LED40.A
- removed net N$52: LED141.A
- removed net N$53: LED55.A
- removed net N$54: LED65.A
- removed net N$55: LED144.A
- removed net N$56: LED8.A
- removed net N$6: U$1.GND@2
- removed net N$78: DECADE-COUNTERA.CLK, U$2.D12
- removed net N$79: DECADE-COUNTERA.RES, U$2.D13
- new net DATA-D11: IC2A.SER, JP2.7
- new net DCLK-D12: IC1A.CLK, JP2.1
- new net LATCH-D9: IC2A.RCK, JP2.6
- new net RESET-D13: IC1A.RES, JP2.2
- new net SRCLK-D10: IC2A.SCK, JP2.5
- net +5V: now also IC1P.VDD, IC2A.SCL, IC2P.VCC, JP2.3; no longer U$1.VIN, U$2.5V
- net GND: now also IC1A.ENA, IC1P.VSS, IC2A.G, IC2P.GND, JP2.4, Q7.E; no longer Q11.E, U$2.GND1
- net N$10: now also R14.1; no longer R4.1
- net N$11: now also R15.1; no longer R5.1
- net N$12: now also R16.1; no longer R6.1
- net N$13: now also R17.1; no longer R7.1
- net N$14: now also R18.1; no longer R8.1
- net N$16: now also LED11.A, LED17.A, LED18.A, LED19.A, LED20.A, R17.2; no longer LED58.A, LED74.A, R7.2
- net N$17: now also LED21.A, LED22.A, LED27.A, LED28.A, LED29.A, LED30.A, R16.2; no longer LED115.A, LED59.A, LED75.A, R6.2
- net N$18: now also LED31.A, LED32.A, LED38.A, LED39.A, LED40.A, R15.2; no longer LED60.A, LED76.A, R5.2
- net N$19: now also LED41.A, LED42.A, LED48.A, LED49.A, LED50.A, R14.2; no longer LED62.A, LED77.A, R4.2
- net N$20: now also LED53.A, LED54.A, LED55.A, LED56.A, LED57.A, LED58.A, LED59.A, LED60.A, R13.2; no longer LED102.A, LED63.A, LED78.A, LED85.A, LED94.A, R3.2
- net N$21: now also LED61.A, LED62.A, LED63.A, LED65.A, LED66.A, LED67.A, R12.2; no longer LED110.A, LED119.A, LED79.A, R2.2
- net N$22: now also LED71.A, LED72.A, LED73.A, LED74.A, LED75.A, LED76.A, LED77.A, LED78.A, LED79.A, R11.2; no longer LED104.A, LED111.A, LED120.A, LED49.A, LED87.A, LED96.A, R1.2
- net N$24: now also LED1.A, LED10.A, LED2.A, LED4.A, LED6.A, LED7.A, LED8.A, LED9.A, R18.2; no longer LED50.A, LED57.A, LED61.A, LED73.A, LED88.A, LED89.A, R8.2
- net N$30: now also LED10.C, LED20.C, LED21.C, LED31.C, LED41.C, LED56.C, LED66.C, LED71.C; no longer LED49.C, LED57.C, LED58.C, LED59.C, LED60.C, LED62.C, LED63.C, LED64.C
- net N$31: now also LED11.C, LED22.C, LED32.C, LED42.C, LED57.C, LED67.C, LED72.C, LED9.C; no longer LED61.C, LED74.C, LED75.C, LED76.C, LED77.C, LED78.C, LED79.C, LED80.C
- net N$32: now also LED60.C, LED70.C, LED75.C; no longer LED102.C, LED104.C
- net N$33: now also LED1.C, LED59.C, LED74.C; no longer LED88.C, LED89.C, LED94.C, LED96.C
- net N$35: now also LED4.C, LED61.C, LED76.C; no longer LED110.C, LED111.C, LED50.C
- net N$37: now also LED30.C, LED62.C, LED77.C, Q7.C; no longer LED115.C, LED119.C, LED120.C, Q8.C
- net N$38: now also LED63.C, LED78.C, Q8.C; no longer LED127.C, LED128.C, Q11.C
- net N$39: now also LED2.C, LED58.C; no longer LED85.C, LED87.C
- net N$48: now also LED49.C, LED64.C, LED79.C; no longer LED133.C, LED135.C, LED136.C
- net N$57: now also LED50.C, LED80.C; no longer LED141.C, LED144.C
- net N$58: now also R1.2; no longer R9.2
- net N$59: now also R2.2; no longer R10.2
- net N$60: now also R3.2; no longer R11.2
- net N$61: now also R4.2; no longer R12.2
- net N$62: now also R5.2; no longer R13.2
- net N$63: now also R6.2; no longer R14.2
- net N$64: now also Q7.B, R7.2; no longer Q8.B, R15.2
- net N$65: now also Q8.B, R8.2; no longer Q11.B, R16.2
- net N$66: now also R9.2; no longer R17.2
- net N$67: now also R10.2; no longer R18.2
- net N$68: now also IC1A.Q0, R1.1; no longer DECADE-COUNTERA.Q0, R9.1
- net N$69: now also IC1A.Q1, R2.1; no longer DECADE-COUNTERA.Q1, R10.1
- net N$7: now also R11.1; no longer R1.1
- net N$70: now also IC1A.Q2, R3.1; no longer DECADE-COUNTERA.Q2, R11.1
- net N$71: now also IC1A.Q3, R4.1; no longer DECADE-COUNTERA.Q3, R12.1
- net N$72: now also IC1A.Q4, R5.1; no longer DECADE-COUNTERA.Q4, R13.1
- net N$73: now also IC1A.Q5, R6.1; no longer DECADE-COUNTERA.Q5, R14.1
- net N$74: now also IC1A.Q6, R7.1; no longer DECADE-COUNTERA.Q6, R15.1
- net N$75: now also IC1A.Q7, R8.1; no longer DECADE-COUNTERA.Q7, R16.1
- net N$76: now also IC1A.Q8, R9.1; no longer DECADE-COUNTERA.Q8, R17.1
- net N$77: now also IC1A.Q9, R10.1; no longer DECADE-COUNTERA.Q9, R18.1
- net N$8: now also R12.1; no longer R2.1
- net N$9: now also R13.1; no longer R3.1
Other:
- moved on the sheet: LED49, LED50, LED57, LED58, LED59, LED60, LED61, LED62, LED63, LED64, LED73, LED74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
